File: Hardware/Sanjeevni_PCB/Sanjeevni_PCB.kicad_pcb (KiCad board)
At the start: 2 copper layers, 0 parts

Commit message: final PCB design KiCad
Parts:
- added C1: 100nF, Capacitor_SMD:C_0402_1005Metric, F.Cu at (116.0, 93.0)
- added C10: 100nF, Capacitor_SMD:C_0402_1005Metric, F.Cu at (114.0, 94.0)
- added C11: 100nF, Capacitor_SMD:C_0402_1005Metric, F.Cu at (111.0, 60.0)
- added C12: 100nF, Capacitor_SMD:C_0402_1005Metric, F.Cu at (88.0, 62.5)
- added C15: 10uF, Capacitor_SMD:C_0402_1005Metric, F.Cu at (111.0, 62.5)
- added C2: 10uF, Capacitor_SMD:C_0805_2012Metric, F.Cu at (119.5, 98.5)
- added C3: 100uF, Capacitor_SMD:C_0805_2012Metric, F.Cu at (119.5, 94.0)
- added C4: 100nF, Capacitor_SMD:C_0402_1005Metric, F.Cu at (116.0, 96.0)
- added C5: 100nF, Capacitor_SMD:C_0402_1005Metric, F.Cu at (109.5, 88.0)
- added C7: 100nF, Capacitor_SMD:C_0402_1005Metric, F.Cu at (120.0, 102.0)
- added C8: 100 µF / 10V, Capacitor_SMD:C_0805_2012Metric, F.Cu at (119.5, 88.5)
- added D1: LED, LED_SMD:LED_0402_1005Metric, F.Cu at (105.5, 81.0)
- added J1: LiPo battery input (3.7V), Connector_JST:JST_PH_S2B-PH-K_1x02_P2.00mm_Horizontal, F.Cu at (83.5, 101.0)
- added J4: Conn_01x03_Socket, Connector_PinSocket_2.00mm:PinSocket_1x03_P2.00mm_Horizontal, F.Cu at (111.5, 100.2)
- added R1: 330, Resistor_SMD:R_0402_1005Metric, F.Cu at (103.0, 81.0)
- added R2: 4.7K, Resistor_SMD:R_0402_1005Metric, F.Cu at (121.0, 73.5)
- added R3: 10K, Resistor_SMD:R_0402_1005Metric, F.Cu at (112.0, 71.0)
- added R4: 10K, Resistor_SMD:R_0402_1005Metric, F.Cu at (86.5, 85.0)
- added R5: 20K, Resistor_SMD:R_0402_1005Metric, F.Cu at (88.0, 91.5)
- added R6: 4.7K, Resistor_SMD:R_0402_1005Metric, F.Cu at (117.0, 76.0)
- added R7: 10K, Resistor_SMD:R_0402_1005Metric, F.Cu at (88.0, 60.0)
- added R8: 10K, Resistor_SMD:R_0402_1005Metric, F.Cu at (111.0, 75.0)
- added RV1: 10K, Potentiometer_THT:Potentiometer_Bourns_3296W_Vertical, F.Cu at (81.0, 88.5)
- added SW1: EN / RESET button, Button_Switch_SMD:SW_SPST_CK_RS282G05A3, F.Cu at (82.0, 63.0)
- added SW2: BOOT / GPIO0 button, Button_Switch_SMD:SW_SPST_CK_RS282G05A3, F.Cu at (116.5, 63.0)
- added TP1: GND, TestPoint:TestPoint_Pad_1.5x1.5mm, F.Cu at (92.5, 82.5)
- added TP2: 3V3, TestPoint:TestPoint_Pad_1.5x1.5mm, F.Cu at (96.5, 82.5)
- added TP3: RX, TestPoint:TestPoint_Pad_1.5x1.5mm, F.Cu at (100.0, 82.5)
- added TP4: EN, TestPoint:TestPoint_Pad_1.5x1.5mm, F.Cu at (91.5, 87.0)
- added TP5: TX, TestPoint:TestPoint_Pad_1.5x1.5mm, F.Cu at (96.0, 86.5)
- added TP6: IO0, TestPoint:TestPoint_Pad_1.5x1.5mm, F.Cu at (105.0, 85.5)
- added U1: AMS1117-3.3, Package_TO_SOT_SMD:SOT-223-3_TabPin2, F.Cu at (82.5, 77.0)
- added U2: MT3608, Package_TO_SOT_SMD:SOT-23-6, F.Cu at (113.5, 90.0)
- added U3: ADXL343, Package_LGA:LGA-14_3x5mm_P0.8mm_LayoutBorder1x6y, F.Cu at (116.5, 72.0)
- added U4: ESP32-WROOM-32, RF_Module:ESP32-WROOM-32, F.Cu at (99.7, 67.4)
- added U5: DHT11, Sensor:Aosong_DHT11_5.5x12.0_P2.54mm, F.Cu at (111.8, 82.0)
- added U6: MQ-6, Sensor:MQ-6, F.Cu at (96.6, 94.1)
Routing:
- net GND: track 0.00 -> 195.0 mm, vias 0 -> 5
- net +3.3V: track 0.00 -> 160.4 mm, vias 0 -> 8
- net /BAT+: track 0.00 -> 63.0 mm, vias 0 -> 2
- net /OUT: track 0.00 -> 46.3 mm, vias 0 -> 2
- net Net-(C11-Pad2): track 0.00 -> 42.5 mm
- net /EN: track 0.00 -> 39.3 mm
- net Net-(U6-A2): track 0.00 -> 35.5 mm
- net /IO0: track 0.00 -> 25.3 mm
- net Net-(U6-A1): track 0.00 -> 23.7 mm, vias 0 -> 1
- net /SDA: track 0.00 -> 23.0 mm, vias 0 -> 3
- net /RX: track 0.00 -> 22.1 mm, vias 0 -> 2
- net /SCL: track 0.00 -> 18.8 mm, vias 0 -> 2
- net Net-(U6-B1): track 0.00 -> 14.4 mm
- net Net-(U6-B2): track 0.00 -> 12.4 mm
- net Net-(U5-DATA): track 0.00 -> 11.8 mm, vias 0 -> 2
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Other:
- board outline added: 45.5 x 57 mm
