File: Hardware/Sanjeevni_PCB/Sanjeevni_PCB.kicad_sch (KiCad schematic)
At the start: 0 parts

Commit message: update pcb schema
Parts:
- added C1, C11, C12, C13, C14, C15, C16, C4, C5, C6, C7, C9: C, Capacitor_SMD:C_0402_1005Metric, symbol Device:C
- added C2, C3, C8: C_Polarized, Capacitor_SMD:C_0805_2012Metric, symbol Device:C_Polarized
- added D1: LED, LED_SMD:LED_0402_1005Metric, symbol Device:LED
- added J1: Conn_01x02, Connector_JST:JST_PH_S2B-PH-K_1x02_P2.00mm_Horizontal, symbol Connector_Generic:Conn_01x02
- added J2, J3: Conn_01x04, Connector:FanPinHeader_1x04_P2.54mm_Vertical, symbol Connector_Generic:Conn_01x04
- added R1, R2, R3, R4, R5: R, Resistor_SMD:R_0402_1005Metric, symbol Device:R
- added RV1: R_Potentiometer_Trim, Potentiometer_THT:Potentiometer_Bourns_3296W_Vertical, symbol Device:R_Potentiometer_Trim
- added SW1, SW2: SW_Push, Button_Switch_SMD:SW_SPST_CK_RS282G05A3, symbol Switch:SW_Push
- added TP1, TP10, TP11, TP12, TP2, TP3, TP4, TP5, TP6, TP7, TP8, TP9: TestPoint, TestPoint:TestPoint_Pad_1.5x1.5mm, symbol Connector:TestPoint
- added U1: AMS1117-3.3, Package_TO_SOT_SMD:SOT-223-3_TabPin2, symbol Regulator_Linear:AMS1117-3.3
- added U2: MT3608, Package_TO_SOT_SMD:SOT-23-6, symbol Regulator_Switching:MT3608
- added U3: ADXL343, Package_LGA:LGA-14_3x5mm_P0.8mm_LayoutBorder1x6y, symbol Sensor_Motion:ADXL343
- added U4: ESP32-WROOM-32, RF_Module:ESP32-WROOM-32, symbol RF_Module:ESP32-WROOM-32
- added U5: DHT11, Sensor:Aosong_DHT11_5.5x12.0_P2.54mm, symbol Sensor:DHT11
- added U6: MQ-6, Sensor:MQ-6, symbol Sensor_Gas:MQ-6
Connections:
- new net: U3.2 (GND), U3.4 (GND), U3.5 (GND)
- new net: U4.1 (GND), U4.15 (GND), U4.38 (GND), U4.39 (GND)
Other:
- company: (none) -> Sanjeevi
- title: (none) -> Schematic Diagram

Commit message: final PCB design KiCad
Parts:
- removed C13, C14, C16, C6, C9: C, Capacitor_SMD:C_0402_1005Metric, symbol Device:C
- removed J2, J3: Conn_01x04, Connector:FanPinHeader_1x04_P2.54mm_Vertical, symbol Connector_Generic:Conn_01x04
- removed TP10, TP11, TP12, TP7, TP8, TP9: TestPoint, TestPoint:TestPoint_Pad_1.5x1.5mm, symbol Connector:TestPoint
- added C10: 100nF, Capacitor_SMD:C_0402_1005Metric, symbol Device:C
- added J4: Conn_01x03_Socket, Connector_PinSocket_2.00mm:PinSocket_1x03_P2.00mm_Horizontal, symbol Connector:Conn_01x03_Socket
- added R6: 4.7K, Resistor_SMD:R_0402_1005Metric, symbol Device:R
- added R7, R8: 10K, Resistor_SMD:R_0402_1005Metric, symbol Device:R
- C1, C11, C12, C4, C5, C7: value C -> 100nF
- C15: value C -> 10uF
- C2: value C_Polarized -> 10uF
- C3: value C_Polarized -> 100uF
- C8: value C_Polarized -> 100 µF / 10V
- J1: value Conn_01x02 -> LiPo battery input (3.7V)
- R1: value R -> 330
- R2: value R -> 4.7K
- R3, R4: value R -> 10K
- R5: value R -> 20K
- RV1: value R_Potentiometer_Trim -> 10K
- SW1: value SW_Push -> EN / RESET button
- SW2: value SW_Push -> BOOT / GPIO0 button
- TP1: value TestPoint -> GND
- TP2: value TestPoint -> 3V3
- TP3: value TestPoint -> RX
- TP4: value TestPoint -> EN
- TP5: value TestPoint -> TX
- TP6: value TestPoint -> IO0
Connections:
- net +3.3V: now reaches U3.1 (Vdd_I/O)
- net +3.3V: now also C11.1, C2.1, C4.1, C5.1, C7.1, C8.1, R2.2, TP2.1, U1.2 (VO), U3.6 (Vs), U3.7 (~{CS}), U4.2 (VDD), U5.1 (VDD), U6.2 (VH+), R6.2, R7.1, R8.1
- net GND: now reaches U3.12 (SDO/ADDR)
- net GND: now also C1.2, C12.2, C15.2, C3.2, C4.2, C5.2, C7.2, C8.2, J1.2 (Pin_2), R1.2, R4.2, R5.2, SW1.2, SW2.2, TP1.1, U1.1 (GND), U2.2 (GND), U2.3 (FB), U3.2 (GND), U3.4 (GND), U3.5 (GND), U5.4 (GND), U6.5 (VH-), C10.2, J4.2 (Pin_2)
- net SDA: now reaches U3.13 (SDA/SDI/SDIO)
- net SDA: now also R2.1, U4.33 (IO21)
- net SCL: now reaches U3.14 (SCL/SCLK)
- net SCL: now also U4.36 (IO22), R6.1
- net at R1.1: now also D1.1 (K)
- net RX: now reaches TP3.1
- net RX: now also U4.34 (RXD0/IO3)
- net BAT+: now reaches J1.1 (Pin_1)
- net BAT+: now also U1.3 (VI), U2.5 (IN)
- net EN: now reaches TP4.1
- net EN: now also C12.1, SW1.1, U4.3 (EN), R7.2
- net at R4.1: now also U6.1 (B1)
- net at U4.1 (GND), U4.15 (GND), U4.38 (GND)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: now also C11.2, C15.1
- net at U4.24 (IO2): now also D1.2 (A)
- net IO0: now reaches U4.25 (IO0)
- net IO0: now also SW2.1, TP6.1, R8.2
- net DATA: now reaches U4.26 (IO4)
- net DATA: now also R3.1
- net TX: now reaches U4.35 (TXD0/IO1)
- net TX: now also TP5.1
- net OUT: now reaches U4.6 (IO34)
- net OUT: now also J4.3 (Pin_3)
- net A0: now reaches U4.7 (IO35)
- net A0: now also RV1.2
- net at U6.3 (B2): now also R5.1
- net at U6.4 (A2): now also RV1.1
- net at U6.6 (A1): now also RV1.3
- net at C1.1: now also U2.4 (EN)
- net at C2.2: now also C3.1
- net at U5.2 (DATA): now also R3.2
- net VCC: now reaches U2.1 (SW)
- net VCC: now also C10.1, J4.1 (Pin_1)
- no-connect marks 0 -> 27
Other:
- moved on the sheet: C1, C11, C12, C15, C2, C3, C4, C5, C7, C8, D1, J1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
